Commit message: sia20: remove fictitious effort limits.

File: motoman_sia_support/urdf/sia20_macro.xacro (robot description, xacro)
@@ -138,5 +138,5 @@
       <origin xyz="0 0 0.41" rpy="0 0 0"/>
       <axis xyz="0 0 1" />
-      <limit lower="-3.1416" upper="3.1416" effort="100" velocity="2.26" />
+      <limit lower="-3.1416" upper="3.1416" effort="0" velocity="2.26" />
     </joint>
     <joint name="${prefix}joint_l" type="revolute">
@@ -145,5 +145,5 @@
       <origin xyz="0 0 0" rpy="0 0 0"/>
       <axis xyz="0 1 0" />
-      <limit lower="-1.91" upper="1.91" effort="100" velocity="2.26" />
+      <limit lower="-1.91" upper="1.91" effort="0" velocity="2.26" />
     </joint>
     <joint name="${prefix}joint_e" type="revolute">
@@ -152,5 +152,5 @@
       <origin xyz="0 0 0.49" rpy="0 0 0"/>
       <axis xyz="0 0 1" />
-      <limit lower="-2.96" upper="2.96" effort="100" velocity="2.96" />
+      <limit lower="-2.96" upper="2.96" effort="0" velocity="2.96" />
     </joint>
     <joint name="${prefix}joint_u" type="revolute">
@@ -159,5 +159,5 @@
       <origin xyz="0 0 0" rpy="0 0 0"/>
       <axis xyz="0 -1 0" />
-      <limit lower="-2.26" upper="2.26" effort="100" velocity="2.96" />
+      <limit lower="-2.26" upper="2.26" effort="0" velocity="2.96" />
     </joint>
     <joint name="${prefix}joint_r" type="revolute">
@@ -166,5 +166,5 @@
       <origin xyz="0 0 0.420" rpy="0 0 0"/>
       <axis xyz="0 0 -1" />
-      <limit lower="-3.1416" upper="3.1416" effort="100" velocity="3.48" />
+      <limit lower="-3.1416" upper="3.1416" effort="0" velocity="3.48" />
     </joint>
     <joint name="${prefix}joint_b" type="revolute">
@@ -173,5 +173,5 @@
       <origin xyz="0 0 0" rpy="0 0 0"/>
       <axis xyz="0 -1 0" />
-      <limit lower="-1.91" upper="1.91" effort="100" velocity="3.48" />
+      <limit lower="-1.91" upper="1.91" effort="0" velocity="3.48" />
     </joint>
     <joint name="${prefix}joint_t" type="revolute">
@@ -180,5 +180,5 @@
       <origin xyz="0 0 0.18" rpy="0 0 0"/>
       <axis xyz="0 0 -1" />
-      <limit lower="-3.1416" upper="3.1416" effort="100" velocity="6.97" />
+      <limit lower="-3.1416" upper="3.1416" effort="0" velocity="6.97" />
     </joint>
     <joint name="${prefix}link_t-tool0" type="fixed" >
